Commit message: Salad Fingers

File: bin/project/resources/panda_arm_hand.urdf (robot description, URDF)
Before this commit: robot panda_hand, 10 links, 9 joints
Links:
- link leftfinger: geometry collision mesh filename=../../../model/panda/meshes/collision/finger.obj scale=1 1 1.8; visual mesh filename=../../../model/panda/meshes/visual/finger.obj scale=1 1 1.8
- link rightfinger: geometry collision mesh filename=../../../model/panda/meshes/collision/finger.obj scale=1 1 1.8; visual mesh filename=../../../model/panda/meshes/visual/finger.obj scale=1 1 1.8
